File: main_board_optimized.brd (EAGLE design)
At the start: 91 x 66 mm, 49 parts, among them IC1 LT1168ACS8, IC2 LT1168ACS8, IC3 LT1168ACS8, IC4 317EMP, U1 TLC272IP, U2 TLC272IP, U3 TLC272IP

Commit message: Better layout
Parts:
- moved TM6 83.4 mm to (104.5, 31.4)
- moved TM7 75.4 mm to (104.4, 18.4)
- moved TM5 68.9 mm to (73.0, 18.4)
- moved PAD6 68.4 mm to (19.1, 38.0)
- moved R6 67.1 mm to (3.68, 17.1), turned to 90 degrees
- moved PAD25 65.2 mm to (22.6, 37.9)
- moved R8 64.0 mm to (112.5, 18.1), turned to 90 degrees
- moved PAD26 60.6 mm to (26.1, 37.9)
- moved PAD7 56.0 mm to (29.8, 38.0)
- moved R7 54.8 mm to (112.6, 31.1), turned to 90 degrees
- moved R4 48.4 mm to (96.0, 26.9), turned to 90 degrees
- moved IC3 45.0 mm to (89.8, 31.2)
- moved R5 44.2 mm to (3.76, 24.1), turned to 90 degrees
- moved R13 43.9 mm to (81.1, 19.1), turned to 90 degrees
- moved U3 40.0 mm to (94.0, 14.1)
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Routing:
- net VDD: track 164.7 -> 593.6 mm
- net N$6: track 94.3 -> 367.1 mm
- net N$27: track 196.0 -> 462.7 mm
- net N$2: track 159.7 -> 387.2 mm
- net VCC: track 120.0 -> 330.0 mm
- net N$25: track 180.2 -> 382.3 mm
- net N$8: track 79.9 -> 279.7 mm
- net N$11: track 77.8 -> 256.2 mm
- net N$24: track 143.0 -> 319.7 mm
- net N$1: track 83.9 -> 249.6 mm
- net N$32: track 96.3 -> 260.9 mm
- net N$18: track 72.1 -> 232.5 mm
- net N$5: track 128.8 -> 276.6 mm
- net N$9: track 16.2 -> 156.5 mm
- net N$13: track 23.6 -> 160.6 mm
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- added copper zone on layer 16, net N$33
Other:
- board size 91 x 66 mm -> 119 x 65 mm

Commit message: Added stuff
Routing:
- removed copper zone on layer 1, net GND
- removed copper zone on layer 16, net N$33
Other:
- board size 119 x 65 mm -> 119 x 43 mm
Changed lines of the file:
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@@
 <plain>
 <wire x1="0" y1="0" x2="119" y2="0" width="0" layer="20"/>
-<wire x1="119" y1="0" x2="119" y2="65" width="0" layer="20"/>
-<wire x1="119" y1="65" x2="0" y2="65" width="0" layer="20"/>
-<wire x1="0" y1="65" x2="0" y2="0" width="0" layer="20"/>
+<wire x1="119" y1="0" x2="119" y2="43" width="0" layer="20"/>
+<wire x1="119" y1="43" x2="0" y2="43" width="0" layer="20"/>
+<wire x1="0" y1="43" x2="0" y2="0" width="0" layer="20"/>
 </plain>
 <attributes>
@@
 <contactref element="PAD11" pad="1"/>
 <contactref element="PAD10" pad="1"/>
-<polygon width="0.1524" layer="1">
-<vertex x="-5" y="82"/>
-<vertex x="-5" y="-4"/>
-<vertex x="105" y="-4"/>
-<vertex x="105" y="80"/>
-<vertex x="103" y="82"/>
-</polygon>
-<wire x1="104.47" y1="28.5625" x2="112.52" y2="16.648" width="0" layer="19" extent="1-1"/>
-<wire x1="91.725" y1="28.58" x2="104.47" y2="28.5625" width="0" layer="19" extent="1-1"/>
+<wire x1="91.725" y1="28.58" x2="95.87" y2="40.77" width="0" layer="19" extent="1-1"/>
+<wire x1="104.47" y1="28.5625" x2="91.725" y2="28.58" width="0" layer="19" extent="1-1"/>
+<wire x1="112.52" y1="16.648" x2="104.47" y2="28.5625" width="0" layer="19" extent="1-1"/>
 <wire x1="81.12" y1="17.648" x2="91.725" y2="28.58" width="0" layer="19" extent="1-1"/>
+<wire x1="86.39" y1="14.08" x2="81.12" y2="17.648" width="0" layer="19" extent="1-1"/>
+<wire x1="75.22" y1="7" x2="81.12" y2="17.648" width="0" layer="19" extent="1-1"/>
 <wire x1="73.07" y1="27.5625" x2="81.12" y2="17.648" width="0" layer="19" extent="1-1"/>
 <wire x1="61.055" y1="29.31" x2="73.07" y2="27.5625" width="0" layer="19" extent="1-1"/>
-<wire x1="29.77" y1="37.96" x2="61.055" y2="29.31" width="0" layer="19" extent="1-1"/>
+<wire x1="66.92" y1="40.77" x2="61.055" y2="29.31" width="0" layer="19" extent="1-1"/>
 <wire x1="60.87" y1="7" x2="75.22" y2="7" width="0" layer="19" extent="1-1"/>
 <wire x1="56.63" y1="15.08" x2="60.87" y2="7" width="0" layer="19" extent="1-1"/>
 <wire x1="49.12" y1="16.488" x2="56.63" y2="15.08" width="0" layer="19" extent="1-1"/>
-<wire x1="15.44" y1="17.76" x2="20.87" y2="14.08" width="0" layer="19" extent="1-1"/>
-<wire x1="16.21" y1="27.91" x2="15.44" y2="17.76" width="0" layer="19" extent="1-1"/>
+<wire x1="40.4" y1="27.5625" x2="49.12" y2="16.488" width="0" layer="19" extent="1-1"/>
+<wire x1="26.275" y1="28.31" x2="40.4" y2="27.5625" width="0" layer="19" extent="1-1"/>
+<wire x1="16.21" y1="27.91" x2="26.275" y2="28.31" width="0" layer="19" extent="1-1"/>
 <wire x1="9.43" y1="30.5625" x2="16.21" y2="27.91" width="0" layer="19" extent="1-1"/>
-<wire x1="26.275" y1="28.31" x2="16.21" y2="27.91" width="0" layer="19" extent="1-1"/>
-<wire x1="40.4" y1="27.5625" x2="49.12" y2="16.488" width="0" layer="19" extent="1-1"/>
-<wire x1="66.92" y1="40.77" x2="29.77" y2="37.96" width="0" layer="19" extent="1-1"/>
+<wire x1="15.44" y1="17.76" x2="16.21" y2="27.91" width="0" layer="19" extent="1-1"/>
+<wire x1="20.87" y1="14.08" x2="15.44" y2="17.76" width="0" layer="19" extent="1-1"/>
+<wire x1="29.77" y1="37.96" x2="26.275" y2="28.31" width="0" layer="19" extent="1-1"/>
+<wire x1="27.52" y1="6" x2="20.87" y2="14.08" width="0" layer="19" extent="1-1"/>
+<wire x1="9.35" y1="7.56" x2="15.44" y2="17.76" width="0" layer="19" extent="1-1"/>
 </signal>
 <signal name="VCC">
@@
 <via x="55.6456" y="2.9558" extent="1-16" drill="0.508"/>
 </signal>
-<signal name="N$33">
-<polygon width="0.1524" layer="16">
-<vertex x="-1" y="-6"/>
-<vertex x="125" y="-6"/>
-<vertex x="125" y="-4"/>
-<vertex x="125" y="70"/>
-<vertex x="-3" y="70"/>
-<vertex x="-3" y="67"/>
-<vertex x="-3" y="-6"/>
-</polygon>
-</signal>
 </signals>

Commit message: Connections made
Parts:
- moved PAD10 19.0 mm to (94.2, 6.00)
- moved PAD3 19.0 mm to (86.2, 6.00)
- moved PAD1 3.16 mm to (87.4, 37.8)
- moved PAD2 3.16 mm to (91.1, 37.8)
- moved PAD28 3.16 mm to (58.2, 37.9)
- moved PAD29 3.16 mm to (61.9, 37.9)
- moved PAD4 3.16 mm to (83.7, 37.9)
- moved PAD5 3.16 mm to (54.2, 38.0)
- moved PAD8 3.16 mm to (65.9, 37.8)
- moved PAD9 3.16 mm to (94.9, 37.8)
Connections:
- removed net N$17: IC3.3, PAD2.1
- removed net N$25: R12.1, TM4.1, U2.3
- removed net N$3: R2.1, TM2.1, U1.3
- removed net N$32: IC2.2, PAD28.1
- removed net N$5: R3.2, TM3.2
- removed net N$6: IC4.1, R5.1, R6.2
- removed net N$9: IC3.5, U3.1, U3.2
- new net N$33: TM1.1
- new net N$36: PAD2.1
- new net N$37: U1.3
- new net N$44: U3.6
- new net N$46: R6.2
- new net N$47: IC4.1
- new net N$49: R2.2
- new net N$50: R7.2
- new net N$54: PAD4.1
- new net N$57: R7.1
- new net N$59: U3.3
- new net N$62: R8.2
- new net N$64: R9.2
- new net N$73: R1.2
- new net N$75: R2.1
- new net N$77: R3.2
- new net N$86: U2.3
- new net N$89: R14.2
- new net N$90: IC2.2
- net N$1: no longer R1.2
- net N$10: no longer TM1.1
- net N$11: no longer R7.1, U3.3
- net N$12: no longer R9.2
- net N$13: no longer R8.2
- net N$14: no longer R9.1
- net N$15: no longer IC3.6
- net N$18: no longer IC3.2
- net N$2: no longer TM3.3
- net N$21: no longer PAD26.1
- net N$22: no longer PAD25.1
- net N$23: no longer R11.2
- net N$24: no longer R11.1
- net N$27: no longer R13.2
- net N$28: no longer R14.2
- net N$7: no longer R4.2, U3.7
- net N$8: no longer R4.1, U3.6
- net VCC: no longer IC3.7, U3.8
- net VDD: no longer PAD4.1, PAD5.1, PAD6.1, R12.2, R2.2, R5.2, R7.2
Routing:
- net VDD: track 593.6 -> 5.56 mm, vias 2 -> 0
- net N$27: track 462.7 -> 0.00 mm, vias 1 -> 0
- net N$25: track 382.3 -> 0.00 mm, vias 2 -> 0
- net N$2: track 387.2 -> 9.70 mm, vias 3 -> 0
- net N$6: track 367.1 -> 0.00 mm, vias 4 -> 0
- net N$3: track 312.6 -> 0.00 mm, vias 1 -> 0
- net N$24: track 319.7 -> 12.2 mm, vias 2 -> 0
- net N$8: track 279.7 -> 0.00 mm
- net N$5: track 276.6 -> 0.00 mm, vias 1 -> 0
- net N$32: track 260.9 -> 0.00 mm, vias 1 -> 0
- net N$11: track 256.2 -> 0.00 mm, vias 2 -> 0
- net N$1: track 249.6 -> 16.1 mm, vias 1 -> 0
- net N$18: track 232.5 -> 0.00 mm, vias 3 -> 0
- net N$17: track 217.6 -> 0.00 mm, vias 2 -> 0
- net N$23: track 232.3 -> 17.4 mm, vias 1 -> 0
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- added copper zone on layer 16, net GND

Commit message: Re-doing main board. Use this
Parts:
- moved U2 7.00 mm to (57.2, 15.1)
- moved R7 6.08 mm to (106.6, 30.1)
- moved TM6 6.08 mm to (98.5, 30.4)
- moved R8 6.00 mm to (106.5, 18.1)
- moved TM7 6.00 mm to (98.4, 18.4)
- moved R11 5.39 mm to (60.3, 26.1)
- moved R4 5.10 mm to (91.0, 25.9)
- moved IC2 5.00 mm to (54.1, 31.9)
- moved R12 5.00 mm to (76.2, 30.1)
- moved R13 5.00 mm to (76.1, 19.1)
- moved R14 5.00 mm to (48.1, 31.1)
- moved R2 5.00 mm to (44.2, 30.9)
- moved TM4 5.00 mm to (68.1, 30.4)
- moved TM5 5.00 mm to (68.0, 18.4)
- moved U3 4.12 mm to (90.0, 13.1)
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Routing:
- net VCC: track 126.4 -> 0.00 mm, vias 1 -> 0
- net GND: track 82.2 -> 0.00 mm, vias 1 -> 0
- net N$20: track 41.6 -> 0.00 mm
- net N$26: track 27.0 -> 0.00 mm
- net N$16: track 22.6 -> 0.00 mm
- net N$30: track 22.1 -> 0.00 mm, vias 1 -> 0
- net N$4: track 17.4 -> 0.00 mm
- net N$23: track 17.4 -> 0.00 mm
- net N$1: track 16.1 -> 0.00 mm
- net N$24: track 12.2 -> 0.00 mm
- net N$2: track 9.70 -> 0.00 mm
- net N$31: track 9.60 -> 0.00 mm
- net N$29: track 6.59 -> 0.00 mm
- net N$19: track 5.85 -> 0.00 mm
- net VDD: track 5.56 -> 0.00 mm
Other:
- board size 119 x 43 mm -> 110 x 43 mm
